Commit message: made some xacros for modularity

File: description/robot.urdf.xacro (robot description, xacro)
@@ -3,5 +3,9 @@
     <xacro:arg name="use_ros2_control" default="true"/>
     <xacro:arg name="sim_mode" default="false"/>
-    <xacro:include filename="robot_core.xacro" />
+    <xacro:include filename="robot_core_2wd.xacro" />
+    <!-- <xacro:include filename="velodyne.xacro" /> -->
+    <xacro:include filename="imu.xacro" />
+    <xacro:include filename="rgb_camera.xacro" />
+    <xacro:include filename="face.xacro" />
     <xacro:if value="$(arg use_ros2_control)">
         <xacro:include filename="ros2_control_2wd.xacro" />
@@ -10,10 +14,10 @@
         <xacro:include filename="gazebo_control.xacro" />
     </xacro:unless>
-    <xacro:include filename="velodyne.xacro" />
     <xacro:velodyne parent_prefix="chassis" frame_prefix="velodyne">
         <origin xyz="0.122 0 0.122" rpy="0 0 0"/>
     </xacro:velodyne>
-    <xacro:include filename="camera.xacro" />
+    <xacro:imu parent_prefix="chassis" frame_prefix="imu">
+        <origin xyz="0.0 0 0.05" rpy="0 0 0"/>
+    </xacro:imu>
     <!-- <xacro:include filename="depth_camera.xacro" /> -->
-    <xacro:include filename="face.xacro" />
 </robot>

File: description/velodyne.xacro (robot description, xacro)
@@ -8,14 +8,4 @@
                 <inertia ixx="0.000908059425" ixy="0" ixz="0" iyy="0.000908059425" iyz="0" izz="0.0011049624"/>
             </inertial>
-            <visual>
-                <!-- <geometry>
-                    <mesh filename="package://velodyne_description/meshes/VLP16_base_1.dae"/>
-                </geometry> -->
-            </visual>
-            <visual>
-                <!-- <geometry>
-                    <mesh filename="package://velodyne_description/meshes/VLP16_base_2.dae"/>
-                </geometry> -->
-            </visual>
             <collision>
                 <origin rpy="0 0 0" xyz="0 0 0.03585"/>
@@ -32,5 +22,8 @@
             </inertial>
             <visual>
-                <origin xyz="0 0 -0.0377"/>
+                <origin xyz="0 0 0.01"/>
+                    <geometry>
+                        <cylinder radius="0.05" length="0.1"/>
+                    </geometry>
                 <!-- <geometry>
                     <mesh filename="package://velodyne_description/meshes/VLP16_scan.dae"/>
@@ -49,46 +42,43 @@
             <child link="velodyne"/>
         </joint>
-        <!-- <gazebo reference="${frame_prefix}_base_link">
-            <material>Gazebo/Yellow</material>
-        </gazebo> -->
         <gazebo reference="velodyne_base_link" >
             <sensor name='velodyne-VLP16' type='ray'>
-            <visualize>0</visualize>
-            <update_rate>10</update_rate>
-            <ray>
-            <scan>
-                <horizontal>
-                <samples>440</samples>
-                <resolution>1</resolution>
-                <min_angle>-3.14159</min_angle>
-                <max_angle>3.14159</max_angle>
-                </horizontal>
-                <vertical>
-                <samples>16</samples>
-                <resolution>1</resolution>
-                <min_angle>-0.261799</min_angle>
-                <max_angle>0.261799</max_angle>
-                </vertical>
-            </scan>
-            <range>
-                <min>0.3</min>
-                <max>131</max>
-                <resolution>0.001</resolution>
-            </range>
-            <noise>
-                <type>gaussian</type>
-                <mean>0</mean>
-                <stddev>0</stddev>
-            </noise>
-            </ray>
-            <plugin name='gazebo_ros_laser_controller' filename='libgazebo_ros_velodyne_laser.so'>
-            <topicName>/points_raw</topicName>
-            <frameName>velodyne</frameName>
-            <min_range>0.9</min_range>
-            <max_range>130.0</max_range>
-            <gaussianNoise>0.008</gaussianNoise>
-            </plugin>
-            <pose>0 0 -0.4377 3.14159 0 3.14159</pose>
-        </sensor>
+                <visualize>1</visualize>
+                <update_rate>10</update_rate>
+                <ray>
+                <scan>
+                    <horizontal>
+                    <samples>440</samples>
+                    <resolution>1</resolution>
+                    <min_angle>-3.14159</min_angle>
+                    <max_angle>3.14159</max_angle>
+                    </horizontal>
+                    <vertical>
+                    <samples>16</samples>
+                    <resolution>1</resolution>
+                    <min_angle>-0.261799</min_angle>
+                    <max_angle>0.261799</max_angle>
+                    </vertical>
+                </scan>
+                <range>
+                    <min>0.3</min>
+                    <max>131</max>
+                    <resolution>0.001</resolution>
+                </range>
+                <noise>
+                    <type>gaussian</type>
+                    <mean>0</mean>
+                    <stddev>0</stddev>
+                </noise>
+                </ray>
+                <plugin name='gazebo_ros_laser_controller' filename='libgazebo_ros_velodyne_laser.so'>
+                    <topicName>/points_raw</topicName>
+                    <frameName>velodyne</frameName>
+                    <min_range>0.9</min_range>
+                    <max_range>130.0</max_range>
+                    <gaussianNoise>0.008</gaussianNoise>
+                </plugin>
+                <pose>0 0 -0.4377 3.14159 0 3.14159</pose>
+            </sensor>
         </gazebo>
     </xacro:macro>

Commit message: complete a fundamental pkg

File: description/robot.urdf.xacro (robot description, xacro)
@@ -14,8 +14,8 @@
         <xacro:include filename="gazebo_control.xacro" />
     </xacro:unless>
-    <xacro:velodyne parent_prefix="chassis" frame_prefix="velodyne">
-        <origin xyz="0.122 0 0.122" rpy="0 0 0"/>
+    <xacro:velodyne parent_prefix="base_link" frame_prefix="velodyne">
+        <origin xyz="-0.122 0 0.138" rpy="0 0 0"/>
     </xacro:velodyne>
-    <xacro:imu parent_prefix="chassis" frame_prefix="imu">
+    <xacro:imu parent_prefix="base_link" frame_prefix="imu">
         <origin xyz="0.0 0 0.05" rpy="0 0 0"/>
     </xacro:imu>

File: description/velodyne.xacro (robot description, xacro)
@@ -24,9 +24,6 @@
                 <origin xyz="0 0 0.01"/>
                     <geometry>
-                        <cylinder radius="0.05" length="0.1"/>
+                        <cylinder radius="0.05" length="0.08"/>
                     </geometry>
-                <!-- <geometry>
-                    <mesh filename="package://velodyne_description/meshes/VLP16_scan.dae"/>
-                </geometry> -->
             </visual>
         </link>
@@ -42,5 +39,5 @@
             <child link="velodyne"/>
         </joint>
-        <gazebo reference="velodyne_base_link" >
+        <gazebo reference="velodyne" >
             <sensor name='velodyne-VLP16' type='ray'>
                 <visualize>0</visualize>

Commit message: udpated for slam

File: description/robot.urdf.xacro (robot description, xacro)
@@ -14,9 +14,9 @@
         <xacro:include filename="gazebo_control.xacro" />
     </xacro:unless>
-    <xacro:velodyne parent_prefix="base_link" frame_prefix="velodyne">
-        <origin xyz="-0.122 0 0.138" rpy="0 0 0"/>
+    <xacro:velodyne parent_prefix="base_footprint" frame_prefix="velodyne">
+        <origin xyz="0.0 0 0.05" rpy="0 0 0"/>
     </xacro:velodyne>
-    <xacro:imu parent_prefix="base_link" frame_prefix="imu">
-        <origin xyz="0.0 0 0.05" rpy="0 0 0"/>
+    <xacro:imu parent_prefix="base_footprint" frame_prefix="imu">
+        <origin xyz="0.0 0 0.05377" rpy="0 0 0"/>
     </xacro:imu>
     <!-- <xacro:include filename="depth_camera.xacro" /> -->

File: description/robot_core_2wd.xacro (robot description, xacro)
@@ -36,11 +36,11 @@
     </link>
     <!-- BASE_FOOTPRINT LINK -->
-    <!-- <link name="base_footprint">
-    </link> -->
-    <!-- <joint name="base_footprint_joint" type="fixed">
-        <parent link="base_footprint"/>
-        <child link="base_link"/>
+    <link name="base_footprint">
+    </link>
+    <joint name="base_footprint_joint" type="fixed">
+        <parent link="base_link"/>
+        <child link="base_footprint"/>
         <origin xyz="0 0 0" rpy="0 0 0"/>
-    </joint> -->
+    </joint>
     <!-- CHASSIS LINK -->
     <joint name="chassis_joint" type="fixed">
